Commit message: prevent the robot from sudden jump of mode switch

File: src/gantry_robot_moveit_config_sim/config/gantry_robot.ros2_control.xacro (robot description, xacro)
@@ -8,4 +8,11 @@
                 <plugin>mock_components/GenericSystem</plugin>
             </hardware>
+            <joint name="world_to_x_rail">
+                <command_interface name="position"/>
+                <state_interface name="position">
+                  <param name="initial_value">${initial_positions['world_to_x_rail']}</param>
+                </state_interface>
+                <state_interface name="velocity"/>
+            </joint>
             <joint name="joint_1_2">
                 <command_interface name="position"/>

File: src/models/urdf/gantry_robot.xacro (robot description, xacro)
@@ -28,37 +28,25 @@
     <origin xyz="0.4 -0.2 0.6" rpy="1.57 0 -1.57" />
   </joint>
-  <link name="x_rail"/>
-  <joint name="world_to_x_rail" type="fixed">
+  <link name="link1">
+    <visual>
+      <origin xyz="0 0 0" rpy="0 0 0" />
+      <geometry>
+        <mesh filename="package://models/meshes/link1.STL" scale="0.001 0.001 0.001" />
+      </geometry>
+      <material name="grey" />
+    </visual>
+    <collision>
+      <origin xyz="0 0 0" rpy="0 0 0" />
+      <geometry>
+        <mesh filename="package://models/meshes/link1.STL" scale="0.001 0.001 0.001" />
+      </geometry>
+    </collision>
+    <inertial>
+      <mass value="1.0" />
+      <inertia ixx="0.1" ixy="0.0" ixz="0.0" iyy="0.1" iyz="0.0" izz="0.1" />
+    </inertial>
+  </link>
+  <joint name="world_to_link1" type="fixed">
     <parent link="world" />
-    <child link="x_rail" />
-    <origin xyz="0 0 0" rpy="0 0 0" />
-  </joint>
-  <link name="y_rail"/>
-  <joint name="x_rail_to_y_rail" type="fixed">
-    <parent link="x_rail" />
-    <child link="y_rail" />
-    <origin xyz="0 0 0" rpy="0 0 0" />
-  </joint>
-  <link name="link1">
-    <visual>
-      <origin xyz="0 0 0" rpy="0 0 0" />
-      <geometry>
-        <mesh filename="package://models/meshes/link1.STL" scale="0.001 0.001 0.001" />
-      </geometry>
-      <material name="grey" />
-    </visual>
-    <collision>
-      <origin xyz="0 0 0" rpy="0 0 0" />
-      <geometry>
-        <mesh filename="package://models/meshes/link1.STL" scale="0.001 0.001 0.001" />
-      </geometry>
-    </collision>
-    <inertial>
-      <mass value="1.0" />
-      <inertia ixx="0.1" ixy="0.0" ixz="0.0" iyy="0.1" iyz="0.0" izz="0.1" />
-    </inertial>
-  </link>
-  <joint name="y_rail_to_link1" type="fixed">
-    <parent link="y_rail" />
     <child link="link1" />
     <origin xyz="0 0 0.35" rpy="0 0 0" />
@@ -88,5 +76,5 @@
     <origin xyz="0.1 0 0.2" rpy="0 0 0" />
     <axis xyz="0 0 1"/>
-    <limit lower="-0.3" upper="-0.3" velocity="0.5" effort="1000"/>
+    <limit lower="-0.3" upper="0.1" velocity="0.5" effort="1000"/>
   </joint>
   <link name="link3">

Commit message: added a fuzzy pose generator for mtc

File: src/gantry_robot_moveit_config_sim/config/gantry_robot.ros2_control.xacro (robot description, xacro)
@@ -8,5 +8,5 @@
                 <plugin>mock_components/GenericSystem</plugin>
             </hardware>
-            <joint name="world_to_x_rail">
+            <!-- <joint name="world_to_x_rail">
                 <command_interface name="position"/>
                 <state_interface name="position">
@@ -14,5 +14,5 @@
                 </state_interface>
                 <state_interface name="velocity"/>
-            </joint>
+            </joint> -->
             <joint name="joint_1_2">
                 <command_interface name="position"/>
